Commit message: senyun and realsense

File: .generated/marvin_CCS_m6.urdf (robot description, URDF)
Before this commit: robot marvin_robot, 23 links, 22 joints
Links:
- link Base_L: geometry collision mesh filename=C:/Users/willi/Desktop/KM_data_converter/km_data_converter/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; visual mesh filename=C:/Users/willi/Desktop/KM_data_converter/km_data_converter/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
- link Base_R: geometry collision mesh filename=C:/Users/willi/Desktop/KM_data_converter/km_data_converter/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; visual mesh filename=C:/Users/willi/Desktop/KM_data_converter/km_data_converter/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
- link Link1_L: geometry collision mesh filename=C:/Users/willi/Desktop/KM_data_converter/km_data_converter/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; visual mesh filename=C:/Users/willi/Desktop/KM_data_converter/km_data_converter/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
- link Link1_R: geometry collision mesh filename=C:/Users/willi/Desktop/KM_data_converter/km_data_converter/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; visual mesh filename=C:/Users/willi/Desktop/KM_data_converter/km_data_converter/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
- link Link2_L: geometry collision mesh filename=C:/Users/willi/Desktop/KM_data_converter/km_data_converter/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; visual mesh filename=C:/Users/willi/Desktop/KM_data_converter/km_data_converter/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
- link Link2_R: geometry collision mesh filename=C:/Users/willi/Desktop/KM_data_converter/km_data_converter/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; visual mesh filename=C:/Users/willi/Desktop/KM_data_converter/km_data_converter/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
- link Link3_L: geometry collision mesh filename=C:/Users/willi/Desktop/KM_data_converter/km_data_converter/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; visual mesh filename=C:/Users/willi/Desktop/KM_data_converter/km_data_converter/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
- link Link3_R: geometry collision mesh filename=C:/Users/willi/Desktop/KM_data_converter/km_data_converter/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; visual mesh filename=C:/Users/willi/Desktop/KM_data_converter/km_data_converter/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
- link Link4_L: geometry collision mesh filename=C:/Users/willi/Desktop/KM_data_converter/km_data_converter/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; visual mesh filename=C:/Users/willi/Desktop/KM_data_converter/km_data_converter/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
- link Link4_R: geometry collision mesh filename=C:/Users/willi/Desktop/KM_data_converter/km_data_converter/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; visual mesh filename=C:/Users/willi/Desktop/KM_data_converter/km_data_converter/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
- link Link5_L: geometry collision mesh filename=C:/Users/willi/Desktop/KM_data_converter/km_data_converter/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; visual mesh filename=C:/Users/willi/Desktop/KM_data_converter/km_data_converter/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
- link Link5_R: geometry collision mesh filename=C:/Users/willi/Desktop/KM_data_converter/km_data_converter/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; visual mesh filename=C:/Users/willi/Desktop/KM_data_converter/km_data_converter/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
- link Link6_L: geometry collision mesh filename=C:/Users/willi/Desktop/KM_data_converter/km_data_converter/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; visual mesh filename=C:/Users/willi/Desktop/KM_data_converter/km_data_converter/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
- link Link6_R: geometry collision mesh filename=C:/Users/willi/Desktop/KM_data_converter/km_data_converter/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; visual mesh filename=C:/Users/willi/Desktop/KM_data_converter/km_data_converter/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
- link Link7_L: geometry collision mesh filename=C:/Users/willi/Desktop/KM_data_converter/km_data_converter/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; visual mesh filename=C:/Users/willi/Desktop/KM_data_converter/km_data_converter/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
- link Link7_R: geometry collision mesh filename=C:/Users/willi/Desktop/KM_data_converter/km_data_converter/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; visual mesh filename=C:/Users/willi/Desktop/KM_data_converter/km_data_converter/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
- link base_link: geometry collision mesh filename=C:/Users/willi/Desktop/KM_data_converter/km_data_converter/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; visual mesh filename=C:/Users/willi/Desktop/KM_data_converter/km_data_converter/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
